Commit message: bug fix - multiple vehicle scan publish bug fix - add third vehicle

File: src/racecar2.xacro (robot description, xacro)
@@ -16,6 +16,6 @@
     <color rgba="0.2 0.2 0.2 1."/>
   </material>
-  <material name="red">
-    <color rgba="1.0 0.0 0.0 1."/>
+  <material name="green">
+    <color rgba="0.0 1.0 0.0 1.0"/>
   </material>
   <link name="base_link$(arg prefix)">
@@ -25,5 +25,5 @@
         <box size="${wheelbase} ${width} ${height}"/>
       </geometry>
-      <material name="red"/>
+      <material name="green"/>
     </visual>
   </link>
